Commit message: fixed the urdf of the ur robotiq robot

File: physics_block_rearrangement_env/assets/urdf/robots/ur3e_robotiq/ur3e_robotiq_140old.urdf (robot description, URDF)
Before this commit: robot ur3e_robotiq, 24 links, 23 joints
Links:
- removed link robotiq_arg2f_base_link
- added link robotiq_140_base_link, mass 0.22652; collision mesh filename=meshes/robotiq_description/meshes/collision/2f_140/robotiq_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; visual mesh filename=meshes/robotiq_description/meshes/visual/2f_140/robotiq_arg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
- added link robotiq_base_link
- link base_link_inertia: geometry collision mesh filename=package://meshes/ur_description/meshes/ur3e/collision/base.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; visual mesh filename=package://meshes/ur_description/meshes/ur3e/visual/base.dae
- link forearm_link: geometry collision mesh filename=package://meshes/ur_description/meshes/ur3e/collision/forea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; visual mesh filename=package://meshes/ur_description/meshes/ur3e/visual/forearm.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
- link left_inner_finger: geometry collision mesh filename=meshes/robotiq_description/meshes/collision/2f_140/robotiq_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; visual mesh filename=meshes/robotiq_description/meshes/visual/2f_140/robotiq_arg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
- link left_inner_knuckle: geometry collision mesh filename=meshes/robotiq_description/meshes/collision/2f_140/robotiq_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; visual mesh filename=meshes/robotiq_description/meshes/visual/2f_140/robotiq_arg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
- link left_outer_finger: geometry collision mesh filename=meshes/robotiq_description/meshes/collision/2f_140/robotiq_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; visual mesh filename=meshes/robotiq_description/meshes/visual/2f_140/robotiq_arg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
- link left_outer_knuckle: geometry collision mesh filename=meshes/robotiq_description/meshes/collision/2f_140/robotiq_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; visual mesh filename=meshes/robotiq_description/meshes/visual/2f_140/robotiq_arg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
- link right_inner_finger: geometry collision mesh filename=meshes/robotiq_description/meshes/collision/2f_140/robotiq_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; visual mesh filename=meshes/robotiq_description/meshes/visual/2f_140/robotiq_arg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
- link right_inner_knuckle: geometry collision mesh filename=meshes/robotiq_description/meshes/collision/2f_140/robotiq_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; visual mesh filename=meshes/robotiq_description/meshes/visual/2f_140/robotiq_arg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
- link right_outer_finger: geometry collision mesh filename=meshes/robotiq_description/meshes/collision/2f_140/robotiq_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; visual mesh filename=meshes/robotiq_description/meshes/visual/2f_140/robotiq_arg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
- link right_outer_knuckle: geometry collision mesh filename=meshes/robotiq_description/meshes/collision/2f_140/robotiq_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; visual mesh filename=meshes/robotiq_description/meshes/visual/2f_140/robotiq_arg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
- link shoulder_link: geometry collision mesh filename=package://meshes/ur_description/meshes/ur3e/collision/shoul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; visual mesh filename=package://meshes/ur_description/meshes/ur3e/visual/shoulder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
- link upper_arm_link: geometry collision mesh filename=package://meshes/ur_description/meshes/ur3e/collision/upper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; visual mesh filename=package://meshes/ur_description/meshes/ur3e/visual/upperarm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
- link wrist_1_link: geometry collision mesh filename=package://meshes/ur_description/meshes/ur3e/collision/wrist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; visual mesh filename=package://meshes/ur_description/meshes/ur3e/visual/wrist1.d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
- link wrist_2_link: geometry collision mesh filename=package://meshes/ur_description/meshes/ur3e/collision/wrist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; visual mesh filename=package://meshes/ur_description/meshes/ur3e/visual/wrist2.d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
- link wrist_3_link: geometry collision mesh filename=package://meshes/ur_description/meshes/ur3e/collision/wrist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; visual mesh filename=package://meshes/ur_description/meshes/ur3e/visual/wrist3.d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
Joints:
- removed joint tool0_gripper_joint
- added joint robotiq_140_base_joint: type fixed, parent robotiq_base_link, child robotiq_140_base_link, origin xyz=0 0 0 rpy=0 0 0
- added joint robotiq_base_joint: type fixed, parent tool0, child robotiq_base_link, origin xyz=0 0 0 rpy=0 0 1.5707963267948966
- joint finger_joint: parent robotiq_arg2f_base_link -> robotiq_140_base_link
- joint left_inner_knuckle_joint: parent robotiq_arg2f_base_link -> robotiq_140_base_link
- joint right_inner_knuckle_joint: parent robotiq_arg2f_base_link -> robotiq_140_base_link
- joint right_outer_knuckle_joint: parent robotiq_arg2f_base_link -> robotiq_140_base_link
